File: PCB/BAL.kicad_pcb (KiCad board)
At the start: 2 copper layers, 45.7 x 90.2 mm, 14 parts, among them J1 Battery, J2 UART, SW1 SW_Push, SW2 Detecteur, SW3 SW_SPST, SW4 NO/NC, U1 ATmega328P-PU, U2 DHT11, U3 SX1276_package

Commit message: Add files via upload
Parts:
- moved SW4 2.84 mm to (157.5, 69.8), turned to 270 degrees
Routing:
- net Net-(SW2-Pad2): track 12.5 -> 5.08 mm
- net +3V3: track 114.1 -> 111.1 mm
